File: HUDVio/HUDvio.brd (EAGLE design)
At the start: 85 x 54 mm, 1 part, among them U1 ST_STM32F446RET7

Commit message: Started video sheet
Parts:
- added U$1: SOLDER_PAD_1X3, Skyhawkson-Connectors:SOLDER_PAD_1X3_3X2MM
- added U2: (no value), Skyhawkson-ICs:MAXIM_MAX7456EUI+T
- added U3: TVP5150AM1PBSR, Skyhawkson-ICs:TI_PBS_(S-PQFP-G32)
Connections:
- new net AGND: U2.20, U3.3, U3.31, U3.7
- new net AVDD: U2.21, U3.32, U3.4
- new net DGND: U2.4, U3.19
- new net DVDD: U2.3, U3.20
- new net IO_DVDD: U3.10
- new net N$1: U$1.1
- new net N$2: U$1.2
- new net PAD: U2.29
- new net PGND: U2.23
- new net PVDD: U2.24
- new net VID-IN: U$1.3
Changed lines of the file:
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@@
 <attribute name="VALUE" x="-31.9" y="0.89" size="1.27" layer="27"/>
+</element>
+<element name="U2" library="Skyhawkson-ICs" library_urn="urn:adsk.eagle:library:24316599" package="MAXIM_MAX7456EUI+T" package3d_urn="urn:adsk.eagle:package:24316635/3" value="" x="-37" y="8" smashed="yes">
+<attribute name="DKPN" value="(N/A) MAX7456EUI+CT-ND" x="-37" y="8" size="1.778" layer="27" display="off"/>
+<attribute name="NAME" x="-37" y="13.8174" size="1.27" layer="25" align="bottom-center"/>
+<attribute name="VALUE" x="-37" y="2.465" size="1.27" layer="27" align="top-center"/>
+</element>
+<element name="U3" library="Skyhawkson-ICs" library_urn="urn:adsk.eagle:library:24316599" package="TI_PBS_(S-PQFP-G32)" package3d_urn="urn:adsk.eagle:package:26067601/5" value="TVP5150AM1PBSR" x="-46" y="7" smashed="yes">
+<attribute name="DKPN" value="296-17016-1-ND" x="-46" y="7" size="1.778" layer="27" display="off"/>
+<attribute name="NAME" x="-46" y="11.5496" size="1.27" layer="25" align="bottom-center"/>
+<attribute name="VALUE" x="-46" y="2.4504" size="1.27" layer="27" align="top-center"/>
+</element>
+<element name="U$1" library="Skyhawkson-Connectors" library_urn="urn:adsk.eagle:library:23896875" package="SOLDER_PAD_1X3_3X2MM" package3d_urn="urn:adsk.eagle:package:26070999/2" value="SOLDER_PAD_1X3" x="-57" y="5" smashed="yes">
+<attribute name="DKPN" value="N/A" x="-57" y="5" size="1.778" layer="27" display="off"/>
 </element>
 </elements>
@@
 <contactref element="U1" pad="30"/>
 </signal>
+<signal name="DVDD">
+<contactref element="U2" pad="3"/>
+<contactref element="U3" pad="20"/>
+<wire x1="-39.8735" y1="10.925" x2="-42.8046" y2="6.75" width="0" layer="19" extent="1-1"/>
+</signal>
+<signal name="DGND">
+<contactref element="U2" pad="4"/>
+<contactref element="U3" pad="19"/>
+<wire x1="-39.8735" y1="10.275" x2="-42.8046" y2="6.25" width="0" layer="19" extent="1-1"/>
+</signal>
+<signal name="AGND">
+<contactref element="U2" pad="20"/>
+<contactref element="U3" pad="3"/>
+<contactref element="U3" pad="7"/>
+<contactref element="U3" pad="31"/>
+<wire x1="-49.1954" y1="7.75" x2="-49.1954" y2="5.75" width="0" layer="19" extent="1-1"/>
+<wire x1="-47.25" y1="10.1954" x2="-49.1954" y2="7.75" width="0" layer="19" extent="1-1"/>
+<wire x1="-34.1265" y1="7.025" x2="-47.25" y2="10.1954" width="0" layer="19" extent="1-1"/>
+</signal>
+<signal name="AVDD">
+<contactref element="U2" pad="21"/>
+<contactref element="U3" pad="32"/>
+<contactref element="U3" pad="4"/>
+<wire x1="-47.75" y1="10.1954" x2="-49.1954" y2="7.25" width="0" layer="19" extent="1-1"/>
+<wire x1="-34.1265" y1="7.675" x2="-47.75" y2="10.1954" width="0" layer="19" extent="1-1"/>
+</signal>
+<signal name="PGND">
+<contactref element="U2" pad="23"/>
+</signal>
+<signal name="PVDD">
+<contactref element="U2" pad="24"/>
+</signal>
+<signal name="PAD">
+<contactref element="U2" pad="29"/>
+</signal>
+<signal name="IO_DVDD">
+<contactref element="U3" pad="10"/>
+</signal>
+<signal name="N$1">
+<contactref element="U$1" pad="1"/>
+</signal>
+<signal name="N$2">
+<contactref element="U$1" pad="2"/>
+</signal>
+<signal name="VID-IN">
+<contactref element="U$1" pad="3"/>
+</signal>
 </signals>

Commit message: Pre dinner commit
Parts:
- added C1: 1UF_0805, Skyhawkson-Capacitors:KEMET_0805
- added C2, C3: 18PF_0805, Skyhawkson-Capacitors:KEMET_0805
- added D1: (no value), Skyhawkson-LEDs and Optoelectronics:SUNLED_XZXXXXXX45S-9
- added R1, R2: 1K_0603, Skyhawkson-Resistors:0603
- added R3, R4, R5, R6: 75R_0603, Skyhawkson-Resistors:0603
- added U$3: SOLDER_PAD_1X3, Skyhawkson-Connectors:SOLDER_PAD_1X3_3X2MM
- added X1: ABRACON_ABM8-27.000MHZ, Skyhawkson-Miscellaneous:ABRACON_ABM8
- moved U2 34.8 mm to (-64.0, -14.0)
Connections:
- net VID-IN renamed VIDEO-IN
- new net +5V: C1.P$2, D1.P$2, U$1.1, U$3.1, U2.3
- new net BLU: R3.2
- new net CLKIN: C2.P$1, U2.5, X1.1
- new net GRE: R4.2
- new net HSYNC: R1.1, U2.18
- new net MAX7456-CS: U2.8
- new net MISO: U2.11
- new net MOSI: U2.9
- new net N$3: R5.1, R6.2
- new net N$4: D1.P$4, R4.1
- new net N$5: D1.P$3, R3.1
- new net RED: R5.2
- new net SCL: U3.21
- new net SCLK: U2.10
- new net SDA: U3.22
- new net VIDEO-OUT: U$3.3
- new net VSYNC: R2.1, U2.17
- new net XFB: C3.P$1, U2.6, X1.3
- net DGND: no longer U2.4
- net DVDD: no longer U2.3
- net GND: now also C1.P$1, C2.P$2, C3.P$2, U$1.2, U$3.2, U2.4, X1.2, X1.4
- net N$1: now also R1.2, R2.2, U2.19; no longer U$1.1
- net N$2: now also D1.P$1, R6.1; no longer U$1.2
