File: HUDVio/HUDvio.sch (EAGLE design)
At the start: 1 part, among them U1 ST_STM32F446RET7

Commit message: Started video sheet
Parts:
- added U$1: SOLDER_PAD_1X3, Skyhawkson-Connectors:SOLDER_PAD_1X3
- added U2: (no value), Skyhawkson-ICs:MAXIM_MAX7456EUI+T
- added U3: TVP5150AM1PBSR, Skyhawkson-ICs:TVP5150AM1PBSR
Connections:
- new net N$1: U$1.1
- new net N$2: U$1.2
- new net VID-IN: U$1.3
Changed lines of the file:
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@@
 </classes>
 <parts>
-<part name="FRAME1" library="Skyhawkson-Miscellaneous" library_urn="urn:adsk.eagle:library:23798804" deviceset="A4-FRAME" device=""/>
+<part name="PRIMARY_MICROPROCESSOR" library="Skyhawkson-Miscellaneous" library_urn="urn:adsk.eagle:library:23798804" deviceset="A4-FRAME" device=""/>
 <part name="U1" library="Skyhawkson-Microcontrollers and Processors" library_urn="urn:adsk.eagle:library:23501288" deviceset="ST_STM32F446RET7" device="" package3d_urn="urn:adsk.eagle:package:24908249/6"/>
+<part name="VIDEO_HANDLING" library="Skyhawkson-Miscellaneous" library_urn="urn:adsk.eagle:library:23798804" deviceset="A4-FRAME" device=""/>
+<part name="U2" library="Skyhawkson-ICs" library_urn="urn:adsk.eagle:library:24316599" deviceset="MAXIM_MAX7456EUI+T" device="" package3d_urn="urn:adsk.eagle:package:24316635/3"/>
+<part name="U3" library="Skyhawkson-ICs" library_urn="urn:adsk.eagle:library:24316599" deviceset="TVP5150AM1PBSR" device="" package3d_urn="urn:adsk.eagle:package:26067601/5"/>
+<part name="U$1" library="Skyhawkson-Connectors" library_urn="urn:adsk.eagle:library:23896875" deviceset="SOLDER_PAD_1X3" device="" package3d_urn="urn:adsk.eagle:package:26070999/2"/>
 </parts>
 <sheets>
@@
 </plain>
 <instances>
-<instance part="FRAME1" gate="G$1" x="0" y="0" smashed="yes">
+<instance part="PRIMARY_MICROPROCESSOR" gate="G$1" x="0" y="0" smashed="yes">
 <attribute name="DRAWING_NAME" x="217.17" y="15.24" size="2.54" layer="94"/>
 <attribute name="LAST_DATE_TIME" x="217.17" y="10.16" size="2.286" layer="94"/>
@@
 </nets>
 </sheet>
+<sheet>
+<plain>
+</plain>
+<instances>
+<instance part="VIDEO_HANDLING" gate="G$1" x="0" y="0" smashed="yes">
+<attribute name="DRAWING_NAME" x="217.17" y="15.24" size="2.54" layer="94"/>
+<attribute name="LAST_DATE_TIME" x="217.17" y="10.16" size="2.286" layer="94"/>
+<attribute name="SHEET" x="230.505" y="5.08" size="2.54" layer="94"/>
+</instance>
+<instance part="U2" gate="G$1" x="60.96" y="124.46" smashed="yes">
+<attribute name="NAME" x="66.04" y="127.508" size="1.27" layer="95"/>
+<attribute name="VALUE" x="66.04" y="92.202" size="1.27" layer="96"/>
+</instance>
+<instance part="U3" gate="G$1" x="134.62" y="132.08" smashed="yes">
+<attribute name="NAME" x="139.7" y="135.128" size="1.778" layer="95"/>
+<attribute name="VALUE" x="139.7" y="78.994" size="1.778" layer="96"/>
+</instance>
+<instance part="U$1" gate="G$1" x="20.32" y="121.92" smashed="yes" rot="MR0"/>
+</instances>
+<busses>
+</busses>
+<nets>
+<net name="N$1" class="0">
+<segment>
+<pinref part="U$1" gate="G$1" pin="1"/>
+<wire x1="20.32" y1="121.92" x2="33.02" y2="121.92" width="0.1524" layer="91"/>
+<wire x1="33.02" y1="121.92" x2="33.02" y2="127" width="0.1524" layer="91"/>
+</segment>
+</net>
+<net name="N$2" class="0">
+<segment>
+<pinref part="U$1" gate="G$1" pin="2"/>
+<wire x1="20.32" y1="116.84" x2="33.02" y2="116.84" width="0.1524" layer="91"/>
+<wire x1="33.02" y1="116.84" x2="33.02" y2="109.22" width="0.1524" layer="91"/>
+</segment>
+</net>
+<net name="VID-IN" class="0">
+<segment>
+<pinref part="U$1" gate="G$1" pin="3"/>
+<wire x1="20.32" y1="111.76" x2="30.48" y2="111.76" width="0.1524" layer="91"/>
+<label x="22.86" y="111.76" size="1.778" layer="95"/>
+</segment>
+</net>
+</nets>
+</sheet>

Commit message: Pre dinner commit
Parts:
- added C1: 1UF_0805, Skyhawkson-Capacitors:1UF_0805
- added C2, C3: 18PF_0805, Skyhawkson-Capacitors:18PF_0805
- added D1: (no value), Skyhawkson-LEDs and Optoelectronics:SUNLED_XZMDKCBDDG45S-9
- added R1, R2: 1K_0603, Skyhawkson-Resistors:1K_0603
- added R3, R4, R5, R6: 75R_0603, Skyhawkson-Resistors:75R_0603
- added U$3: SOLDER_PAD_1X3, Skyhawkson-Connectors:SOLDER_PAD_1X3
- added X1: ABRACON_ABM8-27.000MHZ, Skyhawkson-Miscellaneous:ABRACON_ABM8-27.000MHZ
- U2: device Skyhawkson-ICs:MAXIM_MAX7456EUI+T -> Skyhawkson-ICs:MAXIM_MAX7456
Connections:
- net VID-IN renamed VIDEO-IN
- new net +5V: C1.2, D1.VCC@2, U$1.1, U$3.1, U2.DVDD@3
- new net BLU: R3.2
- new net CLKIN: C2.1, U2.CLKIN@5, X1.1
- new net GND: C1.1, C2.2, C3.2, U$1.2, U$3.2, U2.DGND@4, X1.2, X1.4
- new net GRE: R4.2
- new net HSYNC: R1.1, U2.!HSYNC!@18
- new net MAX7456-CS: U2.!CS!@8
- new net MISO: U2.SDO@11
- new net MOSI: U2.SDI@9
- new net N$3: R5.1, R6.2
- new net N$4: D1.G@4, R4.1
- new net N$5: D1.B@3, R3.1
- new net RED: R5.2
- new net SCL: U3.SCL@21
- new net SCLK: U2.SCLK@10
- new net SDA: U3.SDA@22
- new net VIDEO-OUT: U$3.3
- new net VSYNC: R2.1, U2.!VSYNC!@17
- new net XFB: C3.1, U2.XFB@6, X1.3
- net N$1: now also R1.2, R2.2, U2.!RESET!@19; no longer U$1.1
- net N$2: now also D1.R@1, R6.1; no longer U$1.2
Other:
- note added: "(2*12pF) - 6pF = 18pF"
- note added: "Calculated for 25mA: 68R for GRE/BLU 120R for RED Using 75R for BOM reduction"
- note added: "LED shines THROUGH PCB from back, using substrate as a diffuser"
- note added: "To Runcam Nano"
- note added: "To Video Transmitter"
- moved on the sheet: U2, U3
